File: Kestrel/Dual_Chip.kicad_sch (KiCad schematic)
At the start: 45 parts, among them J1 Conn_01x02_Pin, J2 Conn_01x02_Pin, J3 Conn_01x02_Pin, Q1 SI2301, SW1 SW_SPDT, U1 TP5100, U2 MT3608

Commit message: values updated in the tp circuit
Parts:
- R10: value R_US -> 1K
- R12, R2, R5, R6, R7: now not fitted
- R14: value R_US -> 34K5
- R15: value R_US -> 4K7
Changed lines of the file:
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@@
 		(in_bom yes)
 		(on_board yes)
-		(dnp no)
+		(dnp yes)
 		(property "Reference" "R7"
 			(at 92.71 82.55 90)
@@
 		(in_bom yes)
 		(on_board yes)
-		(dnp no)
+		(dnp yes)
 		(property "Reference" "R5"
 			(at 68.58 158.75 90)
@@
 		(in_bom yes)
 		(on_board yes)
-		(dnp no)
+		(dnp yes)
 		(property "Reference" "R12"
 			(at 111.76 149.86 90)
@@
 		(in_bom yes)
 		(on_board yes)
-		(dnp no)
+		(dnp yes)
 		(property "Reference" "R6"
 			(at 64.77 154.94 90)
@@
 			)
 		)
-		(property "Value" "R_US"
+		(property "Value" "4K7"
 			(at 203.2 77.4699 0)
 			(effects
@@
 			)
 		)
-		(property "Value" "R_US"
+		(property "Value" "34K5"
 			(at 203.2 67.3099 0)
 			(effects
@@
 			)
 		)
-		(property "Value" "R_US"
+		(property "Value" "1K"
 			(at 104.14 83.82 90)
 			(effects
@@
 		(in_bom yes)
 		(on_board yes)
-		(dnp no)
+		(dnp yes)
 		(property "Reference" "R2"
 			(at 43.18 53.34 90)

Commit message: schematic updated
Parts:
- R14: value 34K5 -> 20K
- R15: value 4K7 -> 2K7
Changed lines of the file:
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@@
 			)
 		)
-		(property "Value" "4K7"
+		(property "Value" "2K7"
 			(at 203.2 77.4699 0)
 			(effects
@@
 			)
 		)
-		(property "Value" "34K5"
+		(property "Value" "20K"
 			(at 203.2 67.3099 0)
 			(effects
